File: kicad/geeps_mk1/geeps_mk1.kicad_pcb (KiCad board)
At the start: 4 copper layers, 90 x 55 mm, 99 parts, among them J1 E2213PS0E, J2 JST-PH 01x02 Male, J3 USB_C_Receptacle_USB2.0, J4 Conn_ARM_JTAG_SWD_10, J5 DM3AT-SF, J6 Conn_01x03_Pin, Q1 30V 2.2A, Q2 20V 4.2A, Q3 20V 4.2A, Q4 2N7002, Q5 20V 4.2A, Q6 2N7002, Q7 20V 4.2A, Q8 2N7002, SW1 SW_Push, SW2 SW_Push, SW3 SW_Push, SW4 SW_Push, SW5 SW_Push, SW6 SW_Push, U1 PA1616S, U2 TP4056, U3 AP2112K-3.3, U4 W25Q128JVS, U5 RP2040, Y1 12.000MHz 18pF

Commit message: GSHPS Rev A
Parts:
- removed the D4 at (114.6, 62.9)
- added C3: 0.1uF, Capacitor_SMD:C_0402_1005Metric, B.Cu at (117.7, 70.7)
- added C4: 0.1uF, Capacitor_SMD:C_0402_1005Metric, B.Cu at (149.6, 65.7)
- added C5: 0.1uF, Capacitor_SMD:C_0402_1005Metric, B.Cu at (149.0, 47.1)
- added C6: 0.1uF, Capacitor_SMD:C_0402_1005Metric, B.Cu at (162.1, 47.0)
- added CR1: DRTR5V0U2SR-7, Package_TO_SOT_SMD:SOT-143, F.Cu at (125.5, 65.0)
- added D5: GREEN, LED_SMD:LED_0603_1608Metric, F.Cu at (184.0, 37.0)
- added GRAPHIC1: Graphic, Custom_Graphic:BirdWithPants_Small_Right, F.Cu at (123.5, 36.0)
- added GRAPHIC2: Graphic, Custom_Graphic:BirdWithPants_Small_Left, F.Cu at (127.5, 36.0)
- added PCB1: PCB, Custom_Graphic:PCB_PN_REV, B.Cu at (199.1, 77.8)
- added R21: 115R, Resistor_SMD:R_0402_1005Metric, B.Cu at (188.1, 38.5)
- R4: renamed from R24; value TBD -> 732R
- R5: renamed from R25; value TBD -> 294R
- U3: renamed from U4; footprint Package_SO:SOIC-8_5.23x5.23mm_P1.27mm -> Custom_Package_SO:SOIC-8_5.23x5.23mm_P1.27mm
- moved J3 2.00 mm to (163.0, 73.5)
- moved R3 1.80 mm to (120.8, 65.5), turned to 0 degrees
- moved R20 0.20 mm to (164.6, 61.7)
- moved SW4 0.14 mm to (191.5, 56.5)
- renumbered C11 to C1, C16 to C10, C17 to C11, C18 to C12, C19 to C13, C20 to C14, C21 to C15, C22 to C16, C23 to C17, C24 to C18, C25 to C19, C12 to C2, C26 to C20, C27 to C21, C28 to C22, C29 to C23, C5 to C24, C4 to C25, C1 to C26, C6 to C27, C7 to C28, C8 to C29, C9 to C30, C3 to C31, C2 to C32, C10 to C33, C30 to C34, C13 to C7, C14 to C8, C15 to C9, D7 to D1, D8 to D2, D5 to D3, D6 to D4, D1 to D6, D2 to D7, D3 to D8, J2 to J1, J3 to J2, J6 to J3, J1 to J5, J5 to J6, Q2 to Q1, Q3 to Q2, Q6 to Q3, Q7 to Q5, Q5 to Q6, Q8 to Q7, Q1 to Q8, R6 to R1, R14 to R10, R13 to R11, R27 to R12, R15 to R13, R26 to R14, R16 to R15, R17 to R16, R18 to R17, R19 to R18, R28 to R19, R8 to R2, R21 to R22, R2 to R23, R22 to R24, R23 to R25, R29 to R26, R3 to R27, R4 to R28, R5 to R29, R7 to R3, R1 to R30, R30 to R31, R9 to R6, R10 to R7, R11 to R8, R12 to R9, SW4 to SW1, SW5 to SW2, SW6 to SW3, SW1 to SW4, SW2 to SW5, SW3 to SW6, U2 to U1, U3 to U2, U5 to U4, U1 to U5
Connections:
- U4 pad 18: unconnected-(U5-GPIO15-Pad18) -> /STATUS_LED
Routing:
- net /STATUS_LED: track 0.00 -> 49.2 mm, vias 0 -> 4
- net VBUS: track 8.74 -> 39.3 mm, vias 8 -> 10
- net +3V3: track 47.7 -> 52.2 mm, vias 26 -> 30
- net Net-(D5-K): track 0.00 -> 4.19 mm, vias 0 -> 1
- net Net-(J2-CC2): track 3.21 -> 5.16 mm
- net /~{BATT_STDBY}: track 97.2 -> 95.4 mm
- net /~{BATT_CHRG}: track 98.5 -> 96.7 mm
- net GND: track 2.40 -> 3.93 mm, vias 86 -> 94
- net /SERVO_PPM: track 24.0 -> 25.4 mm
- net /USB_D-: track 73.0 -> 73.8 mm
- net /USB_D+: track 72.9 -> 73.8 mm
- removed copper zone on F.Cu, net VBUS
Other:
- outline, holes or cut-outs redrawn
- board text added: "+"
- board text added: "+3V3"
- board text added: "1S LIPO"
- board text added: "BOOT"
- board text added: "GND"
- board text added: "Global Scavenger Hunt Positioning System pantsforbirds.com"
- board text added: "POWER"
- board text added: "RESET"
- board text added: "S"
- board text added: "SERVO"
- board text added: "STATUS"
