File: kicad/geeps_mk1/geeps_mk1.kicad_sch (KiCad schematic)
At the start: 83 parts, among them J1 E2213PS0E, J2 JST-PH 01x02 Male, J3 USB_C_Receptacle_USB2.0, J4 Conn_ARM_JTAG_SWD_10, J5 DM3D-SF, Q1 30V 2.2A, Q2 20V 4.2A, Q3 20V 4.2A, Q4 2N7002, Q5 20V 4.2A, SW1 SW_Push, SW2 SW_Push, SW3 SW_Push, SW4 SW_Push, SW5 SW_Push, SW6 SW_Push, U1 PA1616S, U2 TP4056, U3 AP2112K-3.3, U4 W25Q128JVS, U5 RP2040, Y1 12.000MHz 18pF

Commit message: Routing for geeps mk1
Parts:
- added D7: RED, LED_SMD:LED_0603_1608Metric, symbol Device:LED
- added D8: GREEN, LED_SMD:LED_0603_1608Metric, symbol Device:LED
- added H1, H2, H3, H4: MountingHole, Custom_MountingHole:MountingHole_2.7mm_M2.5_Isolated, symbol Mechanical:MountingHole
- added J6: Conn_01x03_Pin, Connector_Molex:Molex_PicoBlade_53261-0371_1x03-1MP_P1.25mm_Horizontal, symbol Connector:Conn_01x03_Pin
- added Q6, Q8: 2N7002, Package_TO_SOT_SMD:SOT-23, symbol Transistor_FET:2N7002
- added Q7: 20V 4.2A, Package_TO_SOT_SMD:SOT-23, symbol Device:Q_PMOS_GSD
- added R24, R25: TBD, Resistor_SMD:R_0402_1005Metric, symbol Device:R_US
- added R26, R28, R29, R30: 10k, Resistor_SMD:R_0402_1005Metric, symbol Device:R_US
- added R27: 0R, Resistor_SMD:R_0402_1005Metric, symbol Device:R_US
- J2: symbol Connector:Conn_01x02_Male -> Connector:Conn_01x02_Pin
- J5: value DM3D-SF -> DM3AT-SF; symbol Connector:Micro_SD_Card -> Connector:Micro_SD_Card_Det_Hirose_DM3AT; MPN DM3D-SF -> DM3AT-SF-PEJM5; Standard Cost 0.94 -> 1.88
- SW1, SW2, SW3, SW4, SW5, SW6: footprint Button_Switch_SMD:SW_SPST_B3U-1000P -> Button_Switch_SMD:SW_SPST_TL3342; MPN B3U-1000P -> TL3342F160QG/TR; Standard Cost 0.62 -> 0.40
- U5: symbol MCU_RaspberryPi:RP2040 -> Custom_MCU:RP2040
Connections:
- net GNDPWR is gone; now on net GND: J3.S1 (SHIELD)
- net +3V3: now also Q7.2 (S), R28.1, R30.1
- net +BATT: no longer SW4.2
- net GND: now also J5.11 (SHIELD), U2.9 (GND), J6.1 (Pin_1), Q6.2 (S), Q8.2 (S), R26.2, R29.2
- net VBUS: now also D7.2 (A), D8.2 (A)
- net ~{BATT_CHRG}: now also R24.2
- net ~{BATT_STDBY}: now also R25.2
- net at C25.1, D6.1 (K), R11.2: now also SW4.2, Q6.3 (D)
- net REG_IN: now reaches C26.1, D5.1 (K), Q3.2 (S), R10.1, U3.1 (VIN)
- net GPS_PPS: now reaches U1.13 (1PPS)
- net GPS_PPS: now also U5.27 (GPIO16)
- net ~{SERVO_ENABLE}: now reaches U5.16 (GPIO13)
- net ~{SERVO_ENABLE}: now also Q7.1 (G), R28.2
- net SERVO_PPM: now reaches U5.17 (GPIO14)
- net SERVO_PPM: now also J6.3 (Pin_3)
- net ~{SD_DETECT}: now reaches U5.28 (GPIO17)
- net ~{SD_DETECT}: now also J5.10 (DET_A), R30.2
- net POHO_CTRL: now reaches U5.36 (GPIO24)
- net POHO_CTRL: now also R27.1
- net ~{BATT_VSENSE_ENABLE}: no longer names the net of Q5.1 (G), R2.2
- net ~{BATT_VSENSE_ENABLE}: now also Q8.3 (D); no longer U5.37 (GPIO25)
- new net: J6.2 (Pin_2), Q7.3 (D)
- new net: D8.1 (K), R25.1
- new net: Q6.1 (G), R26.1, R27.2
- new net: D7.1 (K), R24.1
- new net BATT_VSENSE_ENABLE: Q8.1 (G), R29.1, U5.37 (GPIO25)
- no-connect marks 11 -> 17
Other:
- note added: "Charge Status LEDs"
- note added: "Green LED V_f ="
- note added: "Red LED V_f = 2.2V 3.15mcd/mA"
- note added: "TODO: add POHO_CTRL series resistor"
- note added: "Target Brightness = 12mcd"
- moved on the sheet: C11, C12, C23, C24, C25, C26, C27, D5, D6, J2, PART1, Q2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

Commit message: GSHPS Rev A
Parts:
- removed D4: 9V 1A TVS, Diode_SMD:D_SOD-923, symbol Device:D_Zener
- removed PART1: Part, symbol Custom_Placeholder:Part
- added C3, C4, C5, C6: 0.1uF, Capacitor_SMD:C_0402_1005Metric, symbol Device:C
- added CR1: DRTR5V0U2SR-7, Package_TO_SOT_SMD:SOT-143, symbol Custom_Power_Protection:DRTR5V0U2SR-7
- added D5: GREEN, LED_SMD:LED_0603_1608Metric, symbol Device:LED
- added GRAPHIC1: Graphic, Custom_Graphic:BirdWithPants_Small_Right, symbol Custom_Placeholder:Graphic
- added GRAPHIC2: Graphic, Custom_Graphic:BirdWithPants_Small_Left, symbol Custom_Placeholder:Graphic
- added PCB1: PCB, Custom_Graphic:PCB_PN_REV, symbol Custom_Placeholder:PCB
- added R21: 115R, Resistor_SMD:R_0402_1005Metric, symbol Device:R_US
- R4: renamed from R24; value TBD -> 732R; MPN (none) -> RC0402FR-07732RL; Standard Cost (none) -> 0.01
- R5: renamed from R25; value TBD -> 294R; MPN (none) -> RC0402FR-07294RL; Standard Cost (none) -> 0.01
- U3: renamed from U4; footprint Package_SO:SOIC-8_5.23x5.23mm_P1.27mm -> Custom_Package_SO:SOIC-8_5.23x5.23mm_P1.27mm
- renumbered C11 to C1, C16 to C10, C17 to C11, C18 to C12, C19 to C13, C20 to C14, C21 to C15, C22 to C16, C23 to C17, C24 to C18, C25 to C19, C12 to C2, C26 to C20, C27 to C21, C28 to C22, C29 to C23, C5 to C24, C4 to C25, C1 to C26, C6 to C27, C7 to C28, C8 to C29, C9 to C30, C3 to C31, C2 to C32, C10 to C33, C30 to C34, C13 to C7, C14 to C8, C15 to C9, D7 to D1, D8 to D2, D5 to D3, D6 to D4, D1 to D6, D2 to D7, D3 to D8, J2 to J1, J3 to J2, J6 to J3, J1 to J5, J5 to J6, Q2 to Q1, Q3 to Q2, Q6 to Q3, Q7 to Q5, Q5 to Q6, Q8 to Q7, Q1 to Q8, R6 to R1, R14 to R10, R13 to R11, R27 to R12, R15 to R13, R26 to R14, R16 to R15, R17 to R16, R18 to R17, R19 to R18, R28 to R19, R8 to R2, R21 to R22, R2 to R23, R22 to R24, R23 to R25, R29 to R26, R3 to R27, R4 to R28, R5 to R29, R7 to R3, R1 to R30, R30 to R31, R9 to R6, R10 to R7, R11 to R8, R12 to R9, SW4 to SW1, SW5 to SW2, SW6 to SW3, SW1 to SW4, SW2 to SW5, SW3 to SW6, U2 to U1, U3 to U2, U5 to U4, U1 to U5
Connections:
- net +3V3: now also C3.2, C4.2, C5.2, C6.2
- net GND: now also C3.1, C4.1, C5.1, C6.1, CR1.1 (GND)
- net USB_D+: now also CR1.2 (IO1)
- net USB_D-: now also CR1.3 (IO2)
- net VBUS: now also CR1.4 (Vcc), D5.2 (A)
- net STATUS_LED: now reaches U4.18 (GPIO15)
- net STATUS_LED: now also R21.2
- new net: D5.1 (K), R21.1
- no-connect marks 17 -> 16
Other:
- note added: "Coupling 3V3 to GND to use as high speed reference plane."
- note added: "Green LED V_f = 2.2V 1.25mcd/mA"
- note added: "Servo Connector with Power Switch"
- note added: "Status LED"
- note removed: "Green LED V_f ="
- note removed: "TODO: add POHO_CTRL series resistor"
- moved on the sheet: J2, J3, Q5, R1, R19, R3
