File: kicad/gshps/gshps.kicad_pcb (KiCad board)
At the start: 4 copper layers, 90 x 55 mm, 108 parts, among them J1 JST-PH 01x02 Male, J2 USB_C_Receptacle_USB2.0, J3 Conn_01x03_Pin, J4 Conn_ARM_JTAG_SWD_10, J5 E2213PS0E, J6 DM3AT-SF, Q1 20V 4.2A, Q2 20V 4.2A, Q3 2N7002, Q4 2N7002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

Commit message: Make gshps rev B
Parts:
- added Q9: 20V 4.2A, Package_TO_SOT_SMD:SOT-23, B.Cu at (66.6, 33.7)
- added R32: 10k, Resistor_SMD:R_0402_1005Metric, B.Cu at (69.1, 33.7)
- C1, C18, C2, C32: footprint Capacitor_SMD:C_0603_1608Metric -> Capacitor_SMD:C_0805_2012Metric
- D4: value 20V 1A -> 1N4148
- J5: moved to F.Cu
- R4: value 732R -> 287R
- R5: value 294R -> 115R
- moved D2 83.5 mm to (34.5, 54.2), turned to 180 degrees
- moved PCB1 83.3 mm to (117.2, 62.5)
- moved D7 82.7 mm to (53.3, 36.5)
- moved C31 82.6 mm to (51.4, 36.0)
- moved C2 82.5 mm to (95.6, 32.0)
- moved C12 82.5 mm to (86.5, 48.0)
- moved C13 82.5 mm to (86.5, 44.0)
- moved Q5 82.5 mm to (86.5, 62.9)
- moved R18 82.5 mm to (92.3, 57.5)
- moved R19 82.5 mm to (86.5, 60.4)
- moved SW2 82.5 mm to (97.6, 59.2)
- moved C10 82.5 mm to (81.1, 53.0)
- moved C11 82.5 mm to (75.6, 48.0)
- moved C14 82.5 mm to (81.0, 41.0)
- moved C15 82.5 mm to (77.5, 41.0)
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Connections:
- C24 pad 1: +3V3 -> Net-(Q9-D)
- C25 pad 1: +3V3 -> Net-(Q9-D)
- D1 pad 2: VBUS -> +3V3
- D2 pad 2: VBUS -> +3V3
- D5 pad 2: VBUS -> +3V3
- L1 pad 1: +3V3 -> Net-(Q9-D)
- U4 pad 35: unconnected-(U4-GPIO23-Pad35) -> /~{DISPLAY_ENABLE}
Routing:
- net /~{DISPLAY_ENABLE}: track 0.00 -> 22.3 mm, vias 0 -> 2
- net VBUS: track 39.3 -> 19.8 mm, vias 10 -> 8
- net Net-(Q9-D): track 0.00 -> 10.7 mm
- net Net-(U1-CE): track 15.1 -> 20.7 mm
- net /DISPLAY_D_C: track 60.6 -> 55.1 mm, vias 4 -> 3
- net /DISPLAY_ECSM: track 66.4 -> 60.9 mm, vias 4 -> 3
- net /~{BATT_CHRG}: track 96.7 -> 91.3 mm
- net /DISPLAY_SCK: track 65.3 -> 60.1 mm, vias 4 -> 3
- net /DISPLAY_MOSI: track 66.9 -> 61.9 mm, vias 4 -> 3
- net /~{DISPLAY_RST}: track 53.5 -> 50.4 mm, vias 4 -> 3
- net /~{BATT_STDBY}: track 95.4 -> 92.3 mm
- net /~{DISPLAY_BUSY}: track 51.4 -> 49.3 mm, vias 4 -> 3
- net /DISPLAY_BOOST_CSENSE: track 38.8 -> 37.3 mm, vias 2 -> 3
- net Net-(D2-K): track 2.53 -> 1.20 mm
- net Net-(D1-K): track 2.33 -> 1.20 mm
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Other:
- outline, holes or cut-outs redrawn
- board text added: "0 mm / 0 mm"
- board text added: "0.01mm"
- board text added: "0.035mm (1oz)"
- board text added: "0.092mm"
- board text added: "0.2 mm"
- board text added: "0.4mm"
- board text added: "0.744 mm"
- board text added: "4"
- board text added: "90 mm x 55 mm"
- board text added: "BOARD CHARACTERISTICS"
- board text added: "Board Thickness:"
- board text added: "Board overall dimensions:"
- board text added: "Castellated pads:"
- board text added: "Copper"
- board text added: "Copper Finish:"
- board text added: "Copper Layer Count:"
- board text added: "Core"
- board text added: "Dielectric"
- board text added: "Edge card connectors:"
- board text added: "Impedance Control:"
- board text added: "Layer"
- board text added: "Legend"
- board text added: "Min hole diameter:"
- board text added: "Min track/spacing:"
- board text added: "No"
- board text added: "None"
- board text added: "Paste Mask"
- board text added: "Plated Board Edge:"
- board text added: "Prepreg"
- board text added: "Signal"
- board text added: "Solder Mask"
- board text added: "Thickness"
- board text added: "Total thickness: 0.744mm"

Commit message: Make gshps rev C
Parts:
- D3: value 20V 1A -> 40V 2A; footprint Diode_SMD:D_SOD-123 -> Diode_SMD:D_SOD-123F
- J5: footprint Custom_FFC-FPC:Hirose_FH34SRJ-24S-0.5SH_1x24-1MP_P0.50mm_Horizontal -> Custom_FFC-FPC:Hirose_FH34SRJ-24S-0.5SH_1x24-1MP_P0.50mm_Horizontal_Mirrored; moved to B.Cu
- Q3, Q4, Q7: value 2N7002 -> 30V 2.2A
- R1, R3: value 5.1k -> 5.1k 1%
- R12: value 0R -> 5.1k 1%
- R22: value 10k 1% -> 5.1k 1%
- R24: value 30k 1% -> 10k 1%; footprint Capacitor_SMD:C_0402_1005Metric -> Resistor_SMD:R_0402_1005Metric
- R6: value 1.33k -> 5.1k 1%
- moved R12 17.9 mm to (106.2, 34.4), turned to 0 degrees
- moved C33 16.0 mm to (48.8, 49.5)
- moved D8 10.7 mm to (59.0, 42.5)
- moved C30 10.5 mm to (48.8, 47.0)
- moved R30 8.28 mm to (53.0, 37.0), turned to -90 degrees
- moved C31 7.56 mm to (56.0, 42.0), turned to -90 degrees
- moved C32 7.28 mm to (62.5, 38.5), turned to -90 degrees
- moved L1 6.89 mm to (60.4, 34.2), turned to -90 degrees
- moved C24 6.72 mm to (62.7, 31.5)
- moved D7 6.69 mm to (59.0, 40.0), turned to 0 degrees
- moved C27 6.38 mm to (49.0, 38.3), turned to 0 degrees
- moved C29 5.01 mm to (48.8, 44.5)
- moved D6 4.03 mm to (59.0, 37.5)
- moved C25 4.00 mm to (62.6, 34.0), turned to -90 degrees
- moved C26 3.54 mm to (56.0, 38.0), turned to -90 degrees
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Connections:
- Q3 pad 1: Net-(Q3-G) -> /POHO_CTRL
- R12 pad 1: /POHO_CTRL -> GND
- R12 pad 2: Net-(Q3-G) -> Net-(R12-Pad2)
- R14 pad 1: Net-(Q3-G) -> /POHO_CTRL
- R22 pad 1: Net-(Q6-D) -> /BATT_VSENSE
- R22 pad 2: /BATT_VSENSE -> Net-(Q6-D)
- R6 pad 2: GND -> Net-(R12-Pad2)
Routing:
- net /DISPLAY_BOOST_CSENSE: track 37.3 -> 12.4 mm, vias 3 -> 2
- net GND: track 3.93 -> 23.5 mm, vias 94 -> 108
- net /POHO_CTRL: track 23.3 -> 38.5 mm, vias 2 -> 4
- net Net-(Q9-D): track 10.7 -> 0.00 mm
- net /DISPLAY_BOOST_GATE: track 20.7 -> 11.0 mm, vias 3 -> 0
- net Net-(D6-A): track 9.49 -> 0.00 mm
- net /DISPLAY_MOSI: track 61.9 -> 53.4 mm, vias 3 -> 2
- net /DISPLAY_BOOST_OUT+: track 11.8 -> 20.2 mm, vias 1 -> 0
- net /DISPLAY_D_C: track 55.1 -> 62.8 mm, vias 3 -> 2
- net /DISPLAY_BOOST_OUT-: track 9.55 -> 17.2 mm, vias 1 -> 0
- net Net-(D7-A): track 5.03 -> 0.00 mm
- net /DISPLAY_SCK: track 60.1 -> 56.0 mm, vias 3 -> 2
- net /QSPI_SS: track 40.8 -> 37.1 mm, vias 3 -> 2
- net /~{SD_DETECT}: track 40.8 -> 37.9 mm, vias 4 -> 2
- net /QSPI_SD1: track 15.5 -> 12.9 mm
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- added copper zone on B.Cu, net /DISPLAY_BOOST_CSENSE
- added copper zone on B.Cu, net Net-(D6-A)
- added copper zone on B.Cu, net Net-(D7-A)
- added copper zone on B.Cu, net Net-(Q9-D)
Other:
- outline, holes or cut-outs redrawn
- board text added: "0.0175mm (0.5oz)"
- board text added: "0.709 mm"
- board text added: "For Personal Use Only."
- board text added: "SOLIDWORKS Maker Product."
- board text added: "Total thickness: 0.709mm"
- board text removed: "0"
- board text removed: "0 mm"
- board text removed: "0.01 mm"
- board text removed: "0.02"
- board text removed: "0.035 mm"
- board text removed: "0.11 mm"
- board text removed: "0.4 mm"
- board text removed: "0.744 mm"
- board text removed: "1"
- board text removed: "3.3"
- board text removed: "4.29"
- board text removed: "Black"
- board text removed: "Bottom Silk Screen"
- board text removed: "Bottom Solder Mask"
- board text removed: "Bottom Solder Paste"
- board text removed: "Color"
- board text removed: "Dielectric 1"
- board text removed: "Dielectric 2"
- board text removed: "Dielectric 3"
- board text removed: "Epsilon R"
- board text removed: "Layer Name"
- board text removed: "Loss Tangent"
- board text removed: "Not specified"
- board text removed: "Thickness (mm)"
- board text removed: "Top Silk Screen"
- board text removed: "Top Solder Mask"
- board text removed: "Top Solder Paste"
- board text removed: "Total thickness: 0.744mm"
- board text removed: "White"
- board text removed: "copper"
- board text removed: "core"
- board text removed: "prepreg"
