File: kicad/gshps/gshps.kicad_pcb (KiCad board)
At the start: 4 copper layers, 90 x 55 mm, 110 parts, among them J1 JST-PH 01x02 Male, J2 USB_C_Receptacle_USB2.0, J3 Conn_01x03_Pin, J4 Conn_ARM_JTAG_SWD_10, J5 E2213PS0E, J6 DM3AT-SF, Q1 20V 4.2A, Q2 20V 4.2A, Q3 30V 2.2A, Q4 30V 2.2A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

Commit message: Clean up after proposal
Parts:
- added C35: 0.1uF, Capacitor_SMD:C_0402_1005Metric, B.Cu at (77.1, 54.0)
Routing:
- net /GPS_PPS: track 39.0 -> 40.8 mm
- net /~{RESET}: track 38.1 -> 38.8 mm
- net GND: track 23.5 -> 24.0 mm, vias 108 -> 109
