File: kicad/gshps/gshps.kicad_sch (KiCad schematic)
At the start: 108 parts, among them J1 JST-PH 01x02 Male, J2 USB_C_Receptacle_USB2.0, J3 Conn_01x03_Pin, J4 Conn_ARM_JTAG_SWD_10, J5 E2213PS0E, J6 DM3AT-SF, Q1 20V 4.2A, Q2 20V 4.2A, Q3 2N7002, Q4 2N7002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

Commit message: Make gshps rev B
Parts:
- added Q9: 20V 4.2A, Package_TO_SOT_SMD:SOT-23, symbol Device:Q_PMOS_GSD
- added R32: 10k, Resistor_SMD:R_0402_1005Metric, symbol Device:R_US
- C1, C18, C2, C32: footprint Capacitor_SMD:C_0603_1608Metric -> Capacitor_SMD:C_0805_2012Metric
- CR1: MPN (none) -> DRTR5V0U2SR-7; Standard Cost (none) -> 0.11
- D4: value 20V 1A -> 1N4148; symbol Device:D_Schottky -> Device:D; MPN PMEG2010ER,115 -> (none); Standard Cost 0.11 -> (none)
- J1: MPN (none) -> S2B-PH-K-S(LF)(SN); Standard Cost (none) -> 0.02
- J3: MPN (none) -> 0532610371; Standard Cost (none) -> 0.37
- PCB1: REV REV A -> REV B
- R4: value 732R -> 287R; MPN RC0402FR-07732RL -> RC0402FR-07287RL
- R5: value 294R -> 115R; MPN RC0402FR-07294RL -> RC0402FR-07115RL
Connections:
- net +3V3: now also D1.2 (A), D2.2 (A), D5.2 (A), Q9.2 (S), R32.1; no longer C24.1, C25.1, L1.1
- net VBUS: no longer D1.2 (A), D2.2 (A), D5.2 (A)
- net ~{DISPLAY_ENABLE}: now reaches U4.35 (GPIO23)
- net ~{DISPLAY_ENABLE}: now also Q9.1 (G), R32.2
- new net: C24.1, C25.1, L1.1, Q9.3 (D)
- no-connect marks 16 -> 15
Other:
- company: (none) -> Pants for Birds
- title: (none) -> Global Scavenger Hunt Positioning System
- moved on the sheet: C24, C25, C26, C27, C28, C29, C30, C31, C32, C33, D6, D7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

Commit message: Make gshps rev C
Parts:
- D3: value 20V 1A -> 40V 2A; footprint Diode_SMD:D_SOD-123 -> Diode_SMD:D_SOD-123F; MPN PMEG2010ER,115 -> SS2040FL_R1_00001
- J5: footprint Custom_FFC-FPC:Hirose_FH34SRJ-24S-0.5SH_1x24-1MP_P0.50mm_Horizontal -> Custom_FFC-FPC:Hirose_FH34SRJ-24S-0.5SH_1x24-1MP_P0.50mm_Horizontal_Mirrored
- PCB1: REV REV B -> REV C
- Q3, Q4, Q7: value 2N7002 -> 30V 2.2A; MPN (none) -> DMN3200U-7
- R1, R3: value 5.1k -> 5.1k 1%
- R12: value 0R -> 5.1k 1%
- R22: value 10k 1% -> 5.1k 1%
- R24: value 30k 1% -> 10k 1%; footprint Capacitor_SMD:C_0402_1005Metric -> Resistor_SMD:R_0402_1005Metric
- R6: value 1.33k -> 5.1k 1%
Connections:
- net BATT_VSENSE: now also R22.1; no longer R22.2
- net GND: now also R12.1; no longer R6.2
- net POHO_CTRL: now also Q3.1 (G), R14.1; no longer R12.1
- net at Q6.3 (D): now also R22.2; no longer R22.1
- new net: R12.2, R6.2

Commit message: Fix BOM export
Parts:
- D3: Standard Cost 0.11 -> 0.10
- Q3, Q4, Q7: Standard Cost (none) -> 0.14
Changed lines of the file:
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@@
 			)
 		)
+		(property "Standard Cost" "0.14"
+			(at 254 184.15 0)
+			(effects
+				(font
+					(size 1.27 1.27)
+				)
+				(hide yes)
+			)
+		)
 		(pin "1"
 		)
@@
 			)
 		)
+		(property "Standard Cost" "0.14"
+			(at 425.45 106.68 0)
+			(effects
+				(font
+					(size 1.27 1.27)
+				)
+				(hide yes)
+			)
+		)
 		(pin "1"
 		)
@@
 			)
 		)
+		(property "Standard Cost" "0.14"
+			(at 360.68 100.33 0)
+			(effects
+				(font
+					(size 1.27 1.27)
+				)
+				(hide yes)
+			)
+		)
 		(pin "1"
 		)
@@
 			)
 		)
-		(property "Standard Cost" "0.11"
+		(property "Standard Cost" "0.10"
 			(at 477.52 93.98 0)
 			(effects

Commit message: GSHPS enclosure
Parts:
- H1, H2, H3, H4: now in the parts list
Changed lines of the file:
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@@
 		(unit 1)
 		(exclude_from_sim no)
-		(in_bom no)
+		(in_bom yes)
 		(on_board yes)
 		(dnp no)
@@
 			)
 		)
+		(property "Manufacturer" ""
+			(at 111.76 360.68 0)
+			(effects
+				(font
+					(size 1.27 1.27)
+				)
+				(hide yes)
+			)
+		)
 		(instances
 			(project "gshps"
@@
 		(unit 1)
 		(exclude_from_sim no)
-		(in_bom no)
+		(in_bom yes)
 		(on_board yes)
 		(dnp no)
@@
 			)
 		)
+		(property "Manufacturer" ""
+			(at 111.76 345.44 0)
+			(effects
+				(font
+					(size 1.27 1.27)
+				)
+				(hide yes)
+			)
+		)
 		(instances
 			(project "gshps"
@@
 		(unit 1)
 		(exclude_from_sim no)
-		(in_bom no)
+		(in_bom yes)
 		(on_board yes)
 		(dnp no)
@@
 			)
 		)
+		(property "Manufacturer" ""
+			(at 111.76 355.6 0)
+			(effects
+				(font
+					(size 1.27 1.27)
+				)
+				(hide yes)
+			)
+		)
 		(instances
 			(project "gshps"
@@
 		(unit 1)
 		(exclude_from_sim no)
-		(in_bom no)
+		(in_bom yes)
 		(on_board yes)
 		(dnp no)
@@
 			(at 111.76 350.52 0)
 			(effects
+				(font
+					(size 1.27 1.27)
+				)
+				(hide yes)
+			)
+		)
+		(property "Manufacturer" ""
+			(at 111.76 350.52 0)
+			(effects

Commit message: Clean up after proposal
Parts:
- added C35: 0.1uF, Capacitor_SMD:C_0402_1005Metric, symbol Device:C
- PCB1: REV REV C -> REV D
Connections:
- net GND: now also C35.1
- net ~{RESET}: now also C35.2
Other:
- moved on the sheet: R25, SW3
Changed lines of the file:
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@@
 	(title_block
 		(title "Global Scavenger Hunt Positioning System")
-		(date "2025-02-15")
-		(rev "C")
+		(date "2025-03-12")
+		(rev "D")
 		(company "Pants for Birds")
 	)
@@
 	)
 	(junction
-		(at 29.21 177.8)
+		(at 31.75 167.64)
 		(diameter 0)
 		(color 0 0 0 0)
@@
 	)
 	(junction
+		(at 31.75 180.34)
+		(diameter 0)
+		(color 0 0 0 0)
+	)
+	(junction
 		(at 187.96 73.66)
 		(diameter 0)
@@
 	(wire
 		(pts
+			(xy 44.45 180.34) (xy 44.45 177.8)
+		)
+		(stroke
+			(width 0)
+			(type default)
+		)
+	)
+	(wire
+		(pts
 			(xy 57.15 302.26) (xy 71.12 302.26)
 		)
@@
 	(wire
 		(pts
-			(xy 29.21 177.8) (xy 29.21 179.07)
+			(xy 31.75 167.64) (xy 31.75 168.91)
 		)
 		(stroke
@@
 	(wire
 		(pts
+			(xy 31.75 180.34) (xy 31.75 181.61)
+		)
+		(stroke
+			(width 0)
+			(type default)
+		)
+	)
+	(wire
+		(pts
 			(xy 69.85 320.04) (xy 71.12 320.04)
 		)
@@
 	(wire
 		(pts
-			(xy 39.37 177.8) (xy 29.21 177.8)
+			(xy 31.75 167.64) (xy 44.45 167.64)
 		)
 		(stroke
@@
 	(wire
 		(pts
+			(xy 31.75 180.34) (xy 44.45 180.34)
+		)
+		(stroke
+			(width 0)
+			(type default)
+		)
+	)
+	(wire
+		(pts
 			(xy 287.02 285.75) (xy 302.26 285.75)
 		)
@@
 	(wire
 		(pts
-			(xy 29.21 166.37) (xy 29.21 168.91)
+			(xy 31.75 156.21) (xy 31.75 158.75)
 		)
 		(stroke
@@
 	(wire
 		(pts
+			(xy 44.45 167.64) (xy 44.45 170.18)
+		)
+		(stroke
+			(width 0)
+			(type default)
+		)
+	)
+	(wire
+		(pts
 			(xy 250.19 270.51) (xy 250.19 279.4)
 		)
@@
 	(wire
 		(pts
-			(xy 29.21 176.53) (xy 29.21 177.8)
+			(xy 31.75 166.37) (xy 31.75 167.64)
 		)
 		(stroke
@@
 	(wire
 		(pts
-			(xy 29.21 189.23) (xy 29.21 190.5)
+			(xy 31.75 179.07) (xy 31.75 180.34)
 		)
 		(stroke
@@
 	(text "RESET\nBUTTON"
 		(exclude_from_sim no)
-		(at 17.78 186.69 0)
+		(at 20.32 176.53 0)
 		(effects
 			(font
@@
 	)
 	(label "~{RESET}"
-		(at 39.37 177.8 180)
+		(at 41.91 167.64 180)
 		(fields_autoplaced yes)
 		(effects
@@
 	(symbol
 		(lib_id "power:GND")
-		(at 29.21 190.5 0)
+		(at 31.75 181.61 0)
 		(unit 1)
 		(exclude_from_sim no)
@@
 		(fields_autoplaced yes)
 		(property "Reference" "#PWR046"
-			(at 29.21 196.85 0)
+			(at 31.75 187.96 0)
 			(effects
 				(font
@@
 		)
 		(property "Value" "GND"
-			(at 29.21 195.58 0)
+			(at 31.75 186.69 0)
 			(effects
 				(font
@@
 		)
 		(property "Footprint" ""
-			(at 29.21 190.5 0)
+			(at 31.75 181.61 0)
 			(effects
 				(font
@@
 		)
 		(property "Datasheet" ""
-			(at 29.21 190.5 0)
+			(at 31.75 181.61 0)
 			(effects
 				(font
@@
 		)
 		(property "Description" ""
-			(at 29.21 190.5 0)
+			(at 31.75 181.61 0)
 			(effects
 				(font
@@
 	(symbol
 		(lib_id "power:+3V3")
-		(at 29.21 166.37 0)
+		(at 31.75 156.21 0)
 		(unit 1)
 		(exclude_from_sim no)
@@
 		(fields_autoplaced yes)
 		(property "Reference" "#PWR041"
-			(at 29.21 170.18 0)
+			(at 31.75 160.02 0)
 			(effects
 				(font
@@
 		)
 		(property "Value" "+3V3"
-			(at 29.21 161.29 0)
+			(at 31.75 151.13 0)
 			(effects
 				(font
@@
 		)
 		(property "Footprint" ""
-			(at 29.21 166.37 0)
+			(at 31.75 156.21 0)
 			(effects
 				(font
@@
 		)
 		(property "Datasheet" ""
-			(at 29.21 166.37 0)
+			(at 31.75 156.21 0)
 			(effects
 				(font
@@
 		)
 		(property "Description" ""
-			(at 29.21 166.37 0)
+			(at 31.75 156.21 0)
 			(effects
 				(font
@@
 	)
 	(symbol
+		(lib_id "Device:C")
+		(at 44.45 173.99 180)
+		(unit 1)
+		(exclude_from_sim no)
+		(in_bom yes)
+		(on_board yes)
+		(dnp no)
+		(property "Reference" "C35"
+			(at 48.26 172.7199 0)
+			(effects
+				(font
+					(size 1.27 1.27)
+				)
+				(justify right)
+			)
+		)
+		(property "Value" "0.1uF"
+			(at 45.72 176.53 0)
+			(effects
+				(font
+					(size 1.27 1.27)
+				)
+				(justify right)
+			)
+		)
+		(property "Footprint" "Capacitor_SMD:C_0402_1005Metric"
+			(at 43.4848 170.18 0)
+			(effects
+				(font
+					(size 1.27 1.27)
+				)
+				(hide yes)
+			)
+		)
+		(property "Datasheet" "~"
+			(at 44.45 173.99 0)
+			(effects
+				(font
+					(size 1.27 1.27)
+				)
+				(hide yes)
+			)
+		)
+		(property "Description" ""
+			(at 44.45 173.99 0)
+			(effects
+				(font
+					(size 1.27 1.27)
+				)
+				(hide yes)
+			)
+		)
+		(pin "1"
+		)
+		(pin "2"
+		)
+		(instances
+			(project "gshps"
+				(path "/ab385390-0f63-468b-8489-a2ebd6764c2d"
+					(reference "C35")
+					(unit 1)
+				)
+			)
+		)
+	)
+	(symbol
 		(lib_id "Mechanical:MountingHole")
 		(at 111.76 350.52 0)
@@
 			)
 		)
-		(property "REV" "REV C"
+		(property "REV" "REV D"
 			(at 152.4 349.25 0)
 			(effects
@@
 	(symbol
 		(lib_id "Switch:SW_Push")
-		(at 29.21 184.15 90)
+		(at 31.75 173.99 90)
 		(unit 1)
 		(exclude_from_sim no)
@@
 		(dnp no)
 		(property "Reference" "SW3"
-			(at 30.48 182.8799 90)
+			(at 33.02 172.7199 90)
 			(effects
 				(font
@@
 		)
 		(property "Value" "SW_Push"
-			(at 30.48 185.4199 90)
+			(at 33.02 175.2599 90)
 			(effects
 				(font
@@
 		)
 		(property "Footprint" "Button_Switch_SMD:SW_SPST_TL3342"
-			(at 24.13 184.15 0)
+			(at 26.67 173.99 0)
 			(effects
 				(font
@@
 		)
 		(property "Datasheet" "~"
-			(at 24.13 184.15 0)
+			(at 26.67 173.99 0)
 			(effects
 				(font
@@
 		)
 		(property "Description" ""
-			(at 29.21 184.15 0)
+			(at 31.75 173.99 0)
 			(effects
 				(font
@@
 		)
 		(property "MPN" "TL3342F160QG/TR"
-			(at 29.21 184.15 0)
+			(at 31.75 173.99 0)
 			(effects
 				(font
@@
 		)
 		(property "Standard Cost" "0.40"
-			(at 29.21 184.15 0)
+			(at 31.75 173.99 0)
 			(effects
 				(font
@@
 	(symbol
 		(lib_id "Device:R_US")
-		(at 29.21 172.72 0)
+		(at 31.75 162.56 0)
 		(unit 1)
 		(exclude_from_sim no)
@@
 		(dnp no)
 		(property "Reference" "R25"
-			(at 27.94 171.45 0)
+			(at 30.48 161.29 0)
 			(effects
 				(font
@@
 		)
 		(property "Value" "10k"
-			(at 27.94 173.99 0)
+			(at 30.48 163.83 0)
 			(effects
 				(font
@@
 		)
 		(property "Footprint" "Resistor_SMD:R_0402_1005Metric"
-			(at 30.226 172.974 90)
+			(at 32.766 162.814 90)
 			(effects
 				(font
@@
 		)
 		(property "Datasheet" "~"
-			(at 29.21 172.72 0)
+			(at 31.75 162.56 0)
 			(effects
 				(font
@@
 		)
 		(property "Description" ""
-			(at 29.21 172.72 0)
+			(at 31.75 162.56 0)
 			(effects
 				(font
